Commit message: Task 1: Multi-robot simulation with namespacing

File: xacro/barista_robot_model.urdf.xacro (robot description, xacro)
@@ -2,4 +2,5 @@
 <robot xmlns:xacro="http://www.ros.org/wiki/xacro" name="barista_robot">
 <xacro:arg name="include_laser" default="true"/>
+<xacro:arg name="robot_name" default="rick"/>
 <xacro:include filename="$(find barista_robot_description)/xacro/drive_wheel.xacro" />
 <xacro:include filename="$(find barista_robot_description)/xacro/caster_wheel.xacro" />
@@ -7,4 +8,6 @@
 <xacro:include filename="$(find barista_robot_description)/xacro/cup_holder_tray.xacro" />
 <xacro:include filename="$(find barista_robot_description)/xacro/laser_scanner.xacro" />
+<xacro:include filename="$(find barista_robot_description)/xacro/barista_robot.gazebo.xacro" />
+<xacro:property name="robot_name" value="$(arg robot_name)"/>
 <xacro:property name="body_width" value="0.155"/>
 <xacro:property name="body_radius" value="0.178"/>
@@ -31,5 +34,10 @@
           <cylinder length="${body_width}" radius="${body_radius}"/>
         </geometry>
+        <xacro:if value="${robot_name == 'rick'}">
             <material name="red"/>
+        </xacro:if>
+        <xacro:unless value="${robot_name == 'rick'}">
+            <material name="blue"/>
+        </xacro:unless>
     </visual>
     <collision>
@@ -61,51 +69,10 @@
 <xacro:standoff_rod number="4" material="black" parent="chassis" x="-0.05" y="0.12" z="0.1875" length="0.220" radius="0.01" />
 <!-- Cup Holder tray -->
-<xacro:cup_holder_tray material="red" parent="chassis" x="0" y="0" z="0.3425"/>
+<xacro:cup_holder_tray parent="chassis" x="0" y="0" z="0.3425" robot_name="$(arg robot_name)"/>
+<!-- Laser scan -->
 <xacro:if value="$(arg include_laser)">
-  <xacro:laser_scanner parent="chassis" x="0.1" y="0" z="0.0775" />
+  <xacro:laser_scanner parent="chassis" x="0.1" y="0" z="0.0775" robot_name="$(arg robot_name)" />
 </xacro:if>
 <!-- PLUGINS -->
-  <!-- Joint State Publisher Plugin -->
-  <gazebo>
-    <plugin filename="gz-sim-joint-state-publisher-system"
-            name="gz::sim::systems::JointStatePublisher">
-        <topic>/joint_states</topic>
-        <update_rate>30</update_rate>
-        <!-- Publish the state of these joints -->
-        <joint_name>joint_left_wheel</joint_name>
-        <joint_name>joint_right_wheel</joint_name>
-        <joint_name>front_yaw_joint</joint_name>
-        <joint_name>back_yaw_joint</joint_name>
-        <joint_name>front_roll_joint</joint_name>
-        <joint_name>back_roll_joint</joint_name>
-        <joint_name>front_pitch_joint</joint_name>
-        <joint_name>back_pitch_joint</joint_name>
-    </plugin>
-  </gazebo>
-  <!-- Differential Drive Plugin -->
-  <gazebo>
-    <plugin
-        filename="gz-sim-diff-drive-system"
-        name="gz::sim::systems::DiffDrive">
-        <left_joint>joint_left_wheel</left_joint>
-        <right_joint>joint_right_wheel</right_joint>
-        <wheel_separation>0.310</wheel_separation>
-        <wheel_radius>0.0352</wheel_radius>
-        <topic>/cmd_vel</topic>
-        <publish_odom>true</publish_odom>
-        <publish_odom_tf>true</publish_odom_tf>
-        <publish_wheel_tf>true</publish_wheel_tf>
-        <odom_topic>odom</odom_topic>
-        <tf_topic>tf</tf_topic>
-        <frame_id>odom</frame_id>
-        <child_frame_id>base_link</child_frame_id>
-    </plugin>
-  </gazebo>
-  <gazebo>
-  <plugin
-    filename="gz-sim-sensors-system"
-    name="gz::sim::systems::Sensors">
-    <render_engine>ogre2</render_engine>
-  </plugin>
-</gazebo>
+<xacro:barista_gazebo robot_name="$(arg robot_name)" />
 </robot>

File: xacro/cup_holder_tray.xacro (robot description, xacro)
@@ -4,5 +4,5 @@
 <xacro:property name="tray_radius" value="0.16"/>
 <!-- Cup Holder Tray Macro -->
-  <xacro:macro name="cup_holder_tray" params="material parent x y z">
+  <xacro:macro name="cup_holder_tray" params="parent x y z robot_name">
     <link name="cup_holder_tray">
     <visual>
@@ -11,5 +11,10 @@
           <cylinder length="${tray_height}" radius="${tray_radius}"/>
         </geometry>
-        <material name="${material}"/>
+        <xacro:if value="${robot_name == 'rick'}">
+            <material name="red"/>
+        </xacro:if>
+        <xacro:unless value="${robot_name == 'rick'}">
+            <material name="blue"/>
+        </xacro:unless>
     </visual>
     <collision>

File: xacro/laser_scanner.xacro (robot description, xacro)
@@ -1,5 +1,5 @@
 <?xml version="1.0"?>
 <robot xmlns:xacro="http://www.ros.org/wiki/xacro">
-  <xacro:macro name="laser_scanner" params="parent x y z">
+  <xacro:macro name="laser_scanner" params="parent x y z robot_name">
     <link name="laser_scan_link">
       <visual>
@@ -50,6 +50,6 @@
           </range>
         </ray>
-        <topic>scan</topic>
-        <gz_frame_id>laser_scan_link</gz_frame_id>
+        <topic>${robot_name}/scan</topic>
+        <gz_frame_id>${robot_name}/laser_scan_link</gz_frame_id>
       </sensor>
     </gazebo>
