Commit message: Fix laser scanner ray origin height in Xacro model

File: xacro/laser_scanner.xacro (robot description, xacro)
@@ -4,5 +4,6 @@
     <link name="laser_scan_link">
       <visual>
-        <origin xyz="0 0 0" rpy="0 0 0"/>
+        <!-- Shift mesh down so base rests on chassis -->
+        <origin xyz="0 0 -0.035" rpy="0 0 0"/>
         <geometry>
           <mesh filename="package://barista_robot_description/meshes/slamtec_rplidar_s1.dae"/>
@@ -10,5 +11,5 @@
       </visual>
       <collision>
-        <origin xyz="0 0 0" rpy="0 0 0"/>
+        <origin xyz="0 0 -0.035" rpy="0 0 0"/>
         <geometry>
           <cylinder radius="0.02775" length="0.051"/>
@@ -17,5 +18,5 @@
       <inertial>
         <mass value="0.105"/>
-        <origin rpy="0 0 0" xyz="0 0 0"/>
+        <origin xyz="0 0 -0.035" rpy="0 0 0"/>
         <inertia
             ixx="4.297289e-05" ixy="0.0" ixz="0.0"
@@ -27,9 +28,11 @@
       <parent link="${parent}"/>
       <child link="laser_scan_link"/>
-      <origin xyz="${x} ${y} ${z}" rpy="0 0 0"/>
+      <!-- Elevates the TF origin by 0.035m to align with the lens -->
+      <origin xyz="${x} ${y} ${z + 0.035}" rpy="0 0 0"/>
     </joint>
     <gazebo reference="laser_scan_link">
       <sensor name="lidar" type="gpu_lidar">
-        <pose>0 0 0.035 0 0 0</pose>
+        <!-- Origin matches laser_scan_link TF frame -->
+        <pose>0 0 0 0 0 0</pose>
         <always_on>true</always_on>
         <visualize>true</visualize>
